File: untitled.kicad_sch (KiCad schematic)
At the start: 0 parts

Commit message: Switched to RP2354A and re-routed
Other:
- note removed: "to be added"
Changed lines of the file:
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@@
 	(generator_version "9.0")
 	(paper "A4")
-	(text "to be added\n"
-		(exclude_from_sim no)
-		(at 139.954 98.552 0)
-		(effects
-			(font
-				(size 1.27 1.27)
-			)
-		)
-	)
 )
