File: hardware/osd.kicad_sch (KiCad schematic)
At the start: 18 parts, among them U11 PI3A223ZMEX, U37 GS8052-FR

Commit message: switched to 0201
Parts:
- C10, C3, C49, C61, C64: footprint Capacitor_SMD:C_0402_1005Metric -> Capacitor_SMD:C_0201_0603Metric; LCSC C1525 -> C76939
- R10, R21, R30: footprint Resistor_SMD:R_0402_1005Metric -> Capacitor_SMD:C_0201_0603Metric; LCSC (none) -> C473048
- R18: footprint Resistor_SMD:R_0402_1005Metric -> Capacitor_SMD:C_0201_0603Metric; LCSC (none) -> C473570
- R2, R24: footprint Resistor_SMD:R_0402_1005Metric -> Capacitor_SMD:C_0201_0603Metric; LCSC (none) -> C270365
- R25: footprint Resistor_SMD:R_0402_1005Metric -> Capacitor_SMD:C_0201_0603Metric; LCSC (none) -> C270364
- R27, R32: value 33R -> 30R; footprint Resistor_SMD:R_0402_1005Metric -> Capacitor_SMD:C_0201_0603Metric; LCSC (none) -> C778391
- R33: value 100R -> 75R; footprint Resistor_SMD:R_0402_1005Metric -> Capacitor_SMD:C_0201_0603Metric; LCSC (none) -> C473570
Connections:
- net GND: now also C10.2, C3.2, C64.2; no longer C10.1, C3.1, C64.1
- net OSD_SYNCLVL_PWM: now also R10.1; no longer R21.1
- net OSD_SYNC_IN: now also R25.2; no longer R25.1
- net OSD_VBLACK_PWM: now also R21.1; no longer R10.1
- net VBLACK_FILT: now also C3.1, R21.2; no longer C3.2, R10.2
- net VIDEO_IN: now also R27.2; no longer R27.1
- net VID_IN: now also R27.1; no longer R27.2
- net VWHITE_FILT: now also C64.1; no longer C64.2
- net at R33.2, U37.5 (+): now also R25.1; no longer R25.2
- new net: C10.1, R10.2, U37.6 (-)
