File: hardware/rp2350a.kicad_sch (KiCad schematic)
At the start: 49 parts, among them Q2 DMN1150UFB-7B, Q7 DMN1150UFB-7B, U36 RP2354B_C39843328, U41 TS2306A 240GF MSM 9_C2976675, U42 TXU0101DCKR, X1 XTM25012000JT00351001

Commit message: switched to 0201
Parts:
- removed C70, C72, C75, C76, C78, C79, C80, C81, C82, C83, C84, C85, C86, C87: 100n, Capacitor_SMD:C_0402_1005Metric, symbol Device:C
- removed C71, C77: 4.7uF, Capacitor_SMD:C_0402_1005Metric, symbol Device:C
- removed C74: 20p, Capacitor_SMD:C_0402_1005Metric, symbol Device:C
- removed R46: 100k, Resistor_SMD:R_0402_1005Metric, symbol Device:R
- removed R47, R54: 10k, Resistor_SMD:R_0402_1005Metric, symbol Device:R
- removed R48, R49: 30R, Resistor_SMD:R_0402_1005Metric, symbol Device:R
- removed R51, R52: 5.1k, Resistor_SMD:R_0402_1005Metric, symbol Device:R
- removed U41: TS2306A 240GF MSM 9_C2976675, lib:SW-SMD_4P-L3.0-W2.0-P0.85-LS3.5, symbol lib:TS2306A240GFMSM9_C2976675
- removed U42: TXU0101DCKR, lib:SC-70-6_L2.0-W1.3-P0.65-LS2.1-BL, symbol lib:TXU0101DCKR
- added C27, C28, C29, C30, C31, C42, C43, C44, C50, C51, C52, C53, C54, C56, C65: 100n, Capacitor_SMD:C_0201_0603Metric, symbol Device:C
- added C59: 20p, Capacitor_SMD:C_0201_0603Metric, symbol Device:C
- added C60, C62: 4.7uF, Capacitor_SMD:C_0402_1005Metric, symbol Device:C
- added R35, R36, R44: 10k, Capacitor_SMD:C_0201_0603Metric, symbol Device:R
- added R37, R38: 30R, Capacitor_SMD:C_0201_0603Metric, symbol Device:R
- added R39, R41: 5.1k, Capacitor_SMD:C_0201_0603Metric, symbol Device:R
- added U10: TXU0101DRYR, lib:SON-6_L1.5-W1.0-P0.50-TL, symbol lib:TXU0101DRYR
- added U32: TS2306A 240GF MSM 9_C2976675, lib:SW-SMD_4P-L3.0-W2.0-P0.85-LS3.5, symbol lib:TS2306A240GFMSM9_C2976675
- C73: footprint Capacitor_SMD:C_0402_1005Metric -> Capacitor_SMD:C_0201_0603Metric; LCSC C441742 -> C76923
- D8: footprint lib:SOT-23-6_L2.9-W1.6-P0.95-LS2.8-BL -> Package_TO_SOT_SMD:SOT-666
- R11, R13: footprint Resistor_SMD:R_0402_1005Metric -> Capacitor_SMD:C_0201_0603Metric; LCSC C106235 -> C270365
- R17, R5: footprint Resistor_SMD:R_0402_1005Metric -> Capacitor_SMD:C_0201_0603Metric; LCSC C60491 -> C270364
- R20: footprint Resistor_SMD:R_0402_1005Metric -> Capacitor_SMD:C_0201_0603Metric; LCSC C106235 -> C473048
- R22, R56: footprint Resistor_SMD:R_0402_1005Metric -> Capacitor_SMD:C_0201_0603Metric; LCSC C138007 -> C778391
- R23: footprint Resistor_SMD:R_0402_1005Metric -> Capacitor_SMD:C_0201_0603Metric; LCSC C2909316 -> C270365
- R40: value 10k -> 5.1k; footprint Resistor_SMD:R_0402_1005Metric -> Capacitor_SMD:C_0201_0603Metric; LCSC C2909316 -> C270344
- R42: value 6.8k -> 5.1k; footprint Resistor_SMD:R_0402_1005Metric -> Capacitor_SMD:C_0201_0603Metric; LCSC C105872 -> C270344
- R43: value 6.8k -> 100k; footprint Resistor_SMD:R_0402_1005Metric -> Capacitor_SMD:C_0201_0603Metric; LCSC C2906876 -> C270364
- R55: footprint Resistor_SMD:R_0402_1005Metric -> Capacitor_SMD:C_0201_0603Metric; LCSC C25087 -> C270359
Connections:
- net +1.1V: now also C27.1, C28.1, C29.1
- net +3.3V: now also R42.2, C30.1, C31.1, C42.1, C43.1, C44.1, C50.1, C51.1, C52.1, C53.1, C65.1, R36.1, R41.1, U10.1 (VCCA); no longer R42.1, R43.1
- net +5V: now also C54.2, U10.5 (OE), U10.6 (VCCB)
- net +BATT: now also R43.1
- net ADC_VBAT: now also R43.2, C56.2, R35.2
- net BEEPER: now also R13.2; no longer R13.1
- net D+: now also R38.2
- net D-: now also R37.1
- net GND: now also C27.2, C28.2, C29.2, C30.2, C31.2, C42.2, C43.2, C44.2, C50.2, C51.2, C52.2, C53.2, C54.1, C56.1, C59.1, C60.2, C62.2, C65.2, R35.1, R39.1, U10.2 (GND), U32.1
- net I2C_SCL: now also R41.2; no longer R42.2
- net I2C_SDA: now also R42.1; no longer R43.2
- net LED0: now also R22.1; no longer R22.2
- net LED_STRIP: now also U10.4 (BY)
- net LED_STRIP_L: now also U10.3 (A)
- net XIN: now also C59.2
- net XOUT: now also R23.1; no longer R23.2
- net at C73.2, X1.3: now also R23.2; no longer R23.1
- net at R40.2: now also USB1.A5 (CC1)
- net at U36.75 (QSPI_SS): now also R44.2
- net at U36.67 (USB_DP): now also R38.1
- net at USB1.B5 (CC2): now also R39.2
- net at U36.35 (RUN): now also R36.2
- net at R56.2, U36.61 (VREG_AVDD): now also C62.1
- net at R55.2, U36.59 (ADC_AVDD): now also C60.1
- net at Q7.1 (G), R5.2: now also R13.1; no longer R13.2
- net at D6.2 (A): now also R22.2; no longer R22.1
- net at U36.66 (USB_DM): now also R37.2
- new net: R44.1, U32.2
Other:
- note added: "RP2354B: Larger variant with integrated flash (2MB) and more GPIO"
- note removed: "RP2354B: Larger variant with integrated flash (2MB)"
- moved on the sheet: C73, D6, D8, Q2, Q7, R17, USB1, X1
